File: fdcanhat/indicators.kicad_sch (KiCad schematic)
At the start: 16 parts, among them Q2 MMBT3904, U17 74AHCT1G125

Commit message: ish done with schematics
Changed lines of the file:
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@@
 	(text "BUZZER"
 		(exclude_from_sim no)
-		(at 111.76 39.37 0)
+		(at 74.93 39.37 0)
 		(effects
 			(font

Commit message: board layout done, ready for routing
Parts:
- removed B1: FUET-5030, 0_indicators:BUZ-SMD_FST-5030, symbol 0_indicators:FUET-5030
- removed C101: 1u 50V X7R, 0_capacitor_smd:C_0603_1608Metric, symbol Device:C
- removed D10, D11, D12, D13: SK6812, 0_indicators:LED-SMD_4P-L2.0-W2.0-BR, symbol 0_indicators:SK6812
- removed D7: 1N4148W, Diode_SMD:D_SOD-123, symbol Diode:1N4148W
- removed Q2: MMBT3904, Package_TO_SOT_SMD:SOT-23, symbol Transistor_BJT:MMBT3904
- removed R47: 220R, 0_resistor_smd:R_0402_1005Metric, symbol Device:R
- removed R49: 10k, 0_resistor_smd:R_0402_1005Metric, symbol Device:R
- added D2, D3, D4, D5: SK6812, 0_diodes:LED-SMD_4P-L2.0-W2.0-BR, symbol 0_diodes:SK6812
- renumbered C102 to C37, C10 to C38, C11 to C39, C12 to C40, R50 to R18, U17 to U9
Connections:
- net +5V: now also D2.1 (VDD), D3.1 (VDD), D4.1 (VDD), D5.1 (VDD)
- net ADD_LED_D_0: now also D2.4 (DIN)
- net ADD_LED_D_1: now also D2.2 (DOUT), D3.4 (DIN)
- net ADD_LED_D_2: now also D3.2 (DOUT), D4.4 (DIN)
- net ADD_LED_D_3: now also D4.2 (DOUT), D5.4 (DIN)
- net GND: now also D2.3 (GND), D3.3 (GND), D4.3 (GND), D5.3 (GND)
Other:
- note removed: "BUZZER"
- moved on the sheet: C37, C38, C39, C40, R18, U9

Commit message: almost done
Parts:
- renumbered C37 to C31, C38 to C32, C39 to C33, C40 to C34, D2 to D3, D3 to D4, D4 to D5, D5 to D6, R18 to R14, U9 to U8
