File: fdcanhat/fdcan.kicad_sch (KiCad schematic)
At the start: 19 parts, among them J1 Conn_01x04_Mounting, SW1 SW_SPST, U1 MCP2518FD-xQBB, U2 TJA1051TK-3, Y1 20 MHz

Commit message: ish done with schematics
Parts:
- added C31, C36, C37: 100n 50V X7R, 0_capacitor_smd:C_0402_1005Metric, symbol Device:C
- added C32, C35, C38: 1u 50V X7R, 0_capacitor_smd:C_0603_1608Metric, symbol Device:C
- added C33, C34: 26p 50V X7R, 0_capacitor_smd:C_0402_1005Metric, symbol Device:C
- added C39: 10u 50V X7R, 0_capacitor_smd:C_0603_1608Metric, symbol Device:C
- added J4: GH1.25-4P, symbol 0_connectors:Conn_01x04_Mounting
- added JP2: SolderJumper_2_Open, symbol Jumper:SolderJumper_2_Open
- added R10, R11: 0R, 0_capacitor_smd:C_0805_2012Metric, symbol Device:R
- added R12: 10k, 0_capacitor_smd:C_0402_1005Metric, symbol Device:R
- added R13: 120R, 0_capacitor_smd:C_0402_1005Metric, symbol Device:R
- added SW2: SW_SPST, symbol Switch:SW_SPST
- added U7: MCP2518FD-xQBB, Package_DFN_QFN:DFN-14-1EP_3x4.5mm_P0.65mm_EP1.65x4.25mm, symbol 0_transceivers:MCP2518FD-xQBB
- added U8: TJA1051TK-3, 0_transceivers:HVSON-8-1EP_3x3mm_P0.65mm_EP1.6x2.4mm, symbol 0_transceivers:TJA1051TK-3
- added Y2: 20 MHz, symbol Device:Crystal_GND24
- C1, C5, C6, R3, R4: footprint (none) -> 0_capacitor_smd:C_0402_1005Metric
- C2, C7, C8: footprint (none) -> 0_capacitor_smd:C_0603_1608Metric
- C3, C4: value 1u 50V X7R -> 26p 50V X7R; footprint (none) -> 0_capacitor_smd:C_0402_1005Metric
- C9: value 100n 50V X7R -> 10u 50V X7R; footprint (none) -> 0_capacitor_smd:C_0603_1608Metric
- J1: value Conn_01x04_Mounting -> GH1.25-4P
- R1, R2: footprint (none) -> 0_capacitor_smd:C_0805_2012Metric
Connections:
- net +3V3: now also C31.1, C32.1, C37.1, C38.1, U7.14 (VDD), U8.5 (VIO)
- net +5V: now also C35.1, C36.1, C39.1, J4.1 (Pin_1), U8.3 (VCC)
- net GND: now also C7.2, C31.2, C32.2, C33.2, C34.2, C35.2, C36.2, C37.2, C38.2, C39.2, J4.4 (Pin_4), J4.MP1, J4.MP2, R12.1, U7.15 (VSS), U7.7 (VSS), U8.2 (GND), U8.9 (GND), Y2.2, Y2.4
- net SPI1_MISO: now also U7.12 (SDO/MISO)
- net SPI1_MOSI: now also U7.11 (SDI/MOSI)
- net SPI1_SCK: now also U7.10 (SCK)
- net FDCAN1_L: now reaches J1.3 (Pin_3), R3.1, U2.6 (CANL)
- net FDCAN1_H: now reaches J1.2 (Pin_2), JP1.2 (B), SW1.1 (A), U2.7 (CANH)
- net FDCAN1_TX: now reaches R1.1, U1.1 (TXCAN)
- net FDCAN1_RX: now reaches R2.1, U1.2 (RXCAN)
- net FDCAN1_TX_T: now reaches R1.2, U2.1 (TXD)
- net FDCAN1_RX_T: now reaches R2.2, U2.4 (RXD)
- net FDCAN1_S: now reaches R4.2, U2.8 (S)
- new net: JP2.1 (A), R13.2, SW2.2 (B)
- new net FDCAN2_CS: U7.13 (~{CS})
- new net FDCAN2_H: J4.2 (Pin_2), JP2.2 (B), SW2.1 (A), U8.7 (CANH)
- new net FDCAN2_INT: U7.4 (~{INT})
- new net FDCAN2_L: J4.3 (Pin_3), R13.1, U8.6 (CANL)
- new net FDCAN2_OSC1: C34.1, U7.6 (OSC1), Y2.3
- new net FDCAN2_OSC2: C33.1, U7.5 (OSC2), Y2.1
- new net FDCAN2_RX: R10.1, U7.2 (RXCAN)
- new net FDCAN2_RX_T: R10.2, U8.4 (RXD)
- new net FDCAN2_S: R12.2, U8.8 (S)
- new net FDCAN2_TX: R11.1, U7.1 (TXCAN)
- new net FDCAN2_TX_T: R11.2, U8.1 (TXD)
- no-connect marks 3 -> 6

Commit message: board layout done, ready for routing
Parts:
- C19: renamed from C7; value 1u 50V X7R -> 1u 50V X5R; LCSC (none) -> C15849
- C20: renamed from C5; LCSC (none) -> C307331
- C21: renamed from C6; LCSC (none) -> C307331
- C22: renamed from C8; value 1u 50V X7R -> 1u 50V X5R; LCSC (none) -> C15849
- C23: renamed from C9; value 10u 50V X7R -> 10u 50V X5R; footprint 0_capacitor_smd:C_0603_1608Metric -> 0_capacitor_smd:C_0805_2012Metric; LCSC (none) -> C440198
- C24: renamed from C1; LCSC (none) -> C307331
- C25: renamed from C2; value 1u 50V X7R -> 1u 50V X5R; LCSC (none) -> C15849
- C26: renamed from C3; value 26p 50V X7R -> 20p 50V C0G; LCSC (none) -> C1554
- C27: renamed from C4; value 26p 50V X7R -> 20p 50V C0G; LCSC (none) -> C1554
- C28: renamed from C35; value 1u 50V X7R -> 1u 50V X5R; LCSC (none) -> C15849
- C29: renamed from C36; LCSC (none) -> C307331
- C30: renamed from C37; LCSC (none) -> C307331
- C31: renamed from C38; value 1u 50V X7R -> 1u 50V X5R; LCSC (none) -> C15849
- C32: renamed from C39; value 10u 50V X7R -> 10u 50V X5R; footprint 0_capacitor_smd:C_0603_1608Metric -> 0_capacitor_smd:C_0805_2012Metric; LCSC (none) -> C440198
- C33: renamed from C31; LCSC (none) -> C307331
- C34: renamed from C32; value 1u 50V X7R -> 1u 50V X5R; LCSC (none) -> C15849
- C35: renamed from C33; value 26p 50V X7R -> 20p 50V C0G; LCSC (none) -> C1554
- C36: renamed from C34; value 26p 50V X7R -> 20p 50V C0G; LCSC (none) -> C1554
- J4: renamed from J1; footprint (none) -> 0_connectors:SM04B-GHS-TB-LF-SN; LCSC (none) -> C189895
- J5: renamed from J4; footprint (none) -> 0_connectors:SM04B-GHS-TB-LF-SN; LCSC (none) -> C189895
- JP1, JP2: footprint (none) -> Jumper:SolderJumper-2_P1.3mm_Open_RoundedPad1.0x1.5mm
- R10: renamed from R1; footprint 0_capacitor_smd:C_0805_2012Metric -> 0_resistor_smd:R_0805_2012Metric; LCSC (none) -> C17477
- R11: renamed from R2; footprint 0_capacitor_smd:C_0805_2012Metric -> 0_resistor_smd:R_0805_2012Metric; LCSC (none) -> C17477
- R12: renamed from R3; footprint 0_capacitor_smd:C_0402_1005Metric -> 0_resistor_smd:R_0402_1005Metric; LCSC (none) -> C25079
- R13: renamed from R4; footprint 0_capacitor_smd:C_0402_1005Metric -> 0_resistor_smd:R_0402_1005Metric; LCSC (none) -> C25744
- R14: renamed from R11; footprint 0_capacitor_smd:C_0805_2012Metric -> 0_resistor_smd:R_0805_2012Metric; LCSC (none) -> C17477
- R15: renamed from R10; footprint 0_capacitor_smd:C_0805_2012Metric -> 0_resistor_smd:R_0805_2012Metric; LCSC (none) -> C17477
- R16: renamed from R13; footprint 0_capacitor_smd:C_0402_1005Metric -> 0_resistor_smd:R_0402_1005Metric; LCSC (none) -> C25079
- R17: renamed from R12; footprint 0_capacitor_smd:C_0402_1005Metric -> 0_resistor_smd:R_0402_1005Metric; LCSC (none) -> C25744
- SW1, SW2: footprint (none) -> 0_misc:SW-SMD_DSIC01LSGET; LCSC (none) -> C54948
- U6: renamed from U1; value MCP2518FD-xQBB -> MCP2518FDT; footprint Package_DFN_QFN:DFN-14-1EP_3x4.5mm_P0.65mm_EP1.65x4.25mm -> 0_transceivers:SOIC-14_3.9x8.7mm_P1.27mm; LCSC (none) -> C626758
- U8: renamed from U7; value MCP2518FD-xQBB -> MCP2518FDT; footprint Package_DFN_QFN:DFN-14-1EP_3x4.5mm_P0.65mm_EP1.65x4.25mm -> 0_transceivers:SOIC-14_3.9x8.7mm_P1.27mm; LCSC (none) -> C626758
- Y1, Y2: footprint (none) -> 0_misc:CRYSTAL-SMD_4P-L3.2-W2.5-BL-2
- renumbered U2 to U5, U8 to U7
Connections:
- net FDCAN1_T_J: now reaches JP1.1 (A), R12.2, SW1.2 (B)
- net FDCAN2_T_J: now reaches JP2.1 (A), R16.2, SW2.2 (B)
- net SPI1_MISO renamed SPI0_MISO
- net SPI1_MOSI renamed SPI0_MOSI
- net SPI1_SCK renamed SPI0_SCK

Commit message: almost done
Parts:
- removed C19, C22, C25, C28, C31, C34: 1u 50V X5R, 0_capacitor_smd:C_0603_1608Metric, symbol Device:C
- removed JP1, JP2: SolderJumper_2_Open, Jumper:SolderJumper-2_P1.3mm_Open_RoundedPad1.0x1.5mm, symbol Jumper:SolderJumper_2_Open
- removed R11, R14, R15: 0R, 0_resistor_smd:R_0805_2012Metric, symbol Device:R
- removed R12: 120R, 0_resistor_smd:R_0402_1005Metric, symbol Device:R
- added C17, C24: 1u 25V X7R, 0_capacitor_smd:C_0402_1005Metric, symbol Device:C
- C22: renamed from C26; value 20p 50V C0G -> 27p 50V C0G; LCSC C1554 -> C3889037
- C23: renamed from C27; value 20p 50V C0G -> 27p 50V C0G; LCSC C1554 -> C3889037
- C29: renamed from C35; value 20p 50V C0G -> 27p 50V C0G; LCSC C1554 -> C3889037
- C30: renamed from C36; value 20p 50V C0G -> 27p 50V C0G; LCSC C1554 -> C3889037
- R10: value 0R -> 120R; LCSC C17477 -> C25079
- R12: renamed from R16; footprint 0_resistor_smd:R_0402_1005Metric -> 0_resistor_smd:R_0805_2012Metric
- SW1, SW2: LCSC C54948 -> (none)
- U5: renamed from U6; footprint 0_transceivers:SOIC-14_3.9x8.7mm_P1.27mm -> 0_transceivers:DFN-14-1EP_3x4.5mm_P0.65mm_EP1.65x4.25mm; LCSC C626758 -> C621395
- U7: renamed from U8; footprint 0_transceivers:SOIC-14_3.9x8.7mm_P1.27mm -> 0_transceivers:DFN-14-1EP_3x4.5mm_P0.65mm_EP1.65x4.25mm; LCSC C626758 -> C621395
- renumbered C20 to C18, C21 to C19, C23 to C20, C24 to C21, C29 to C25, C30 to C26, C32 to C27, C33 to C28, R13 to R11, R17 to R13, U5 to U4, U7 to U6
Connections:
- net FDCAN1_RX_T is gone; now on net FDCAN1_RX: U4.4 (RXD)
- net FDCAN1_T_J is gone; now on net FDCAN1_L: SW1.2 (B)
- net FDCAN2_RX_T is gone; now on net FDCAN2_RX: U6.4 (RXD)
- net FDCAN2_TX_T is gone; now on net FDCAN2_TX: U6.1 (TXD)
- net +5V: now also C17.1, C24.1
- net FDCAN1_H: now also J4.3 (Pin_3), R10.1; no longer J4.2 (Pin_2), SW1.1 (A)
- net FDCAN1_L: now also J4.2 (Pin_2); no longer J4.3 (Pin_3)
- net FDCAN1_TX: now also U4.1 (TXD); no longer R10.1
- net FDCAN2_H: now also J5.3 (Pin_3), R12.1; no longer J5.2 (Pin_2), SW2.1 (A)
- net FDCAN2_L: now also J5.2 (Pin_2), SW2.2 (B); no longer J5.3 (Pin_3), R12.1
- net GND: now also C17.2, C24.2
- net FDCAN1_TX_T renamed FDCAN1_T
- net FDCAN1_T: now also SW1.1 (A); no longer U4.1 (TXD)
- net FDCAN2_T_J renamed FDCAN2_T
- net FDCAN2_T: now also SW2.1 (A); no longer SW2.2 (B)
Other:
- moved on the sheet: C18, C21, C25, C28, R12

Commit message: done doublechecking, going for review
Parts:
- removed J4, J5: GH1.25-4P, 0_connectors:SM04B-GHS-TB-LF-SN, symbol 0_connectors:Conn_01x04_Mounting
- added J4, J5: GH1.25-5P, 0_connectors:SM05B-GHS-TB-LF-SN, symbol 0_connectors:Conn_01x05_Mounting
- R10, R12: LCSC C25079 -> C17437
- SW1, SW2: LCSC (none) -> C54948
Connections:
- net +5V: now also J4.1 (Pin_1), J5.1 (Pin_1)
- net FDCAN1_H: now also J4.3 (Pin_3)
- net FDCAN1_L: now also J4.2 (Pin_2)
- net FDCAN2_H: now also J5.3 (Pin_3)
- net FDCAN2_L: now also J5.2 (Pin_2)
- net GND: now also J4.4 (Pin_4), J4.5 (Pin_5), J4.MP1, J4.MP2, J5.4 (Pin_4), J5.5 (Pin_5), J5.MP1, J5.MP2
