File: fdcanhat/misc.kicad_sch (KiCad schematic)
At the start: 7 parts

Commit message: board layout done, ready for routing
Parts:
- removed H1, H2, H3, H4: M3, MountingHole:MountingHole_3.2mm_M3_Pad_Via, symbol Mechanical:MountingHole_Pad_MP
- added H1, H2, H3, H4: MountingHole_Pad, 0_misc:MountingHole_3.2mm_M3_Pad_Via, symbol Mechanical:MountingHole_Pad
Connections:
- net GND: now also H1.1, H2.1, H3.1, H4.1

Commit message: almost done
Parts:
- H1, H2, H3, H4: footprint 0_misc:MountingHole_3.2mm_M3_Pad_Via -> MountingHole:MountingHole_2.7mm_M2.5_Pad_Via

Commit message: ready for last scrut
Other:
- note added: "M2.5 MOUNTING HOLES"
- note removed: "LOGOS AND GRAPHICS"
- note removed: "M3 MOUNTING HOLES"
- moved on the sheet: FID1, FID2, FID3, H1, H2, H3, H4
