File: fdcanhat/power_generation.kicad_sch (KiCad schematic)
At the start: 0 parts

Commit message: ish done with schematics
Parts:
- added C20, C24, C25, C26, C27, C28, C29, C30: 10u 50V X7R, symbol Device:C
- added C21: 100n 50V X7R, symbol Device:C
- added C22: 47p 50V X7R, symbol Device:C
- added C23: 2n7 50V X7R, symbol Device:C
- added L1: 4.7 uH @ 9A, symbol Device:L
- added R23: 33k, symbol Device:R
- added R24: 10k, symbol Device:R
- added R6: 200K, symbol Device:R
- added R7: 119K, symbol Device:R
- added R8: 15k8, symbol Device:R
- added R9: 22k1, symbol Device:R
- added U5: AP64500, 0_power:SO-8-EP, symbol 0_power:AP64500
- added U6: SPX3819, 0_power:SOT-23-5, symbol 0_power:SPX3819
Connections:
- new net: C22.2, R7.1, R9.2, U5.5 (FB)
- new net: R6.2, U5.4 (RT/CLK)
- new net: C23.1, R8.1
- new net: R8.2, U5.6 (COMP)
- new net: C21.1, L1.1, U5.8 (SW)
- new net: C21.2, U5.1 (BST)
- new net +3V3: C29.1, C30.1, U6.5 (VOUT)
- new net +5V: C22.1, C24.1, C25.1, C26.1, C27.1, C28.1, L1.2, R23.2, R7.2, U6.1 (VIN), U6.3 (EN)
- new net +5V_VMON: R23.1, R24.2
- new net +BAT_PROT: C20.1, U5.2 (VIN), U5.3 (EN)
- new net GND: C20.2, C23.2, C24.2, C25.2, C26.2, C27.2, C28.2, C29.2, C30.2, R24.1, R6.1, R9.1, U5.7 (GND), U5.9 (EPAD), U6.2 (GND)
- no-connect marks 0 -> 1
Other:
- note added: "3V3 LOW DROPOUT REGULATOR"
- note added: "5V BUCK CONVERTER"
- title: (none) -> Power Generation

Commit message: board layout done, ready for routing
Parts:
- removed C25, C26: 10u 50V X7R, symbol Device:C
- added C12, C13: 22u 25V X5R, 0_capacitor_smd:C_0805_2012Metric, symbol Device:C
- C10: renamed from C22; value 47p 50V X7R -> 47p 50V C0G; footprint (none) -> 0_capacitor_smd:C_0402_1005Metric; LCSC (none) -> C1567
- C11: renamed from C24; value 10u 50V X7R -> 22u 25V X5R; footprint (none) -> 0_capacitor_smd:C_0805_2012Metric; LCSC (none) -> C45783
- C14: renamed from C23; footprint (none) -> 0_capacitor_smd:C_0402_1005Metric; LCSC (none) -> C106251
- C15: renamed from C28; value 10u 50V X7R -> 10u 50V X5R; footprint (none) -> 0_capacitor_smd:C_0805_2012Metric; LCSC (none) -> C440198
- C16: renamed from C27; value 10u 50V X7R -> 10u 50V X5R; footprint (none) -> 0_capacitor_smd:C_0805_2012Metric; LCSC (none) -> C440198
- C17: renamed from C29; value 10u 50V X7R -> 10u 50V X5R; footprint (none) -> 0_capacitor_smd:C_0805_2012Metric; LCSC (none) -> C440198
- C18: renamed from C30; value 10u 50V X7R -> 10u 50V X5R; footprint (none) -> 0_capacitor_smd:C_0805_2012Metric; LCSC (none) -> C440198
- C8: renamed from C21; footprint (none) -> 0_capacitor_smd:C_0402_1005Metric; LCSC (none) -> C307331
- C9: renamed from C20; value 10u 50V X7R -> 10u 50V X5R; footprint (none) -> 0_capacitor_smd:C_0805_2012Metric; LCSC (none) -> C440198
- L1: value 4.7 uH @ 9A -> 3.3 uH @ 8.5A; footprint (none) -> 0_inductors:IND-SMD_L11.6-W10.1; LCSC (none) -> C167219
- R4: renamed from R23; footprint (none) -> 0_resistor_smd:R_0402_1005Metric; LCSC (none) -> C25779
- R5: renamed from R7; value 119K -> 53k6; footprint (none) -> 0_resistor_smd:R_0402_1005Metric; LCSC (none) -> C53398
- R6: renamed from R24; footprint (none) -> 0_resistor_smd:R_0402_1005Metric; LCSC (none) -> C25744
- R7: renamed from R6; footprint (none) -> 0_resistor_smd:R_0402_1005Metric; LCSC (none) -> C25764
- R8: footprint (none) -> 0_resistor_smd:R_0402_1005Metric; LCSC (none) -> C26956
- R9: value 22k1 -> 10k; footprint (none) -> 0_resistor_smd:R_0402_1005Metric; LCSC (none) -> C25744
- renumbered U5 to U3, U6 to U4
Connections:
- net +5V: now also C12.1, C13.1
- net GND: now also C12.2, C13.2
- net BUCK_FB: now reaches C10.2, R5.1, R9.2, U3.5 (FB)
- net BUCK_CLK: now reaches R7.2, U3.4 (RT/CLK)
- net BUCK_COMP: now reaches R8.2, U3.6 (COMP)
- net BUCK_SW: now reaches C8.1, L1.1, U3.8 (SW)
- net BUCK_BST: now reaches C8.2, U3.1 (BST)
Other:
- moved on the sheet: C14, C8, R7, R8

Commit message: almost done
Parts:
- L1: footprint 0_inductors:IND-SMD_L11.6-W10.1 -> 0_inductors:IND-SMD_L7.0-W6.6
- renumbered C12 to C10, C13 to C11, C14 to C12, C15 to C13, C16 to C14, C17 to C15, C18 to C16, C8 to C6, C9 to C7, C10 to C8, C11 to C9, U3 to U2, U4 to U3

Commit message: done doublechecking, going for review
Changed lines of the file:
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@@
 		)
 	)
-	(text_box "DESIGN:\nHAT+ specs specifies 5.1 V\n\n119K and 22k1 gives 5.11 V"
+	(text_box "DESIGN:\nHAT+ specs specifies 5.1 V\n\n53k6 and 10k gives 5.11 V"
 		(exclude_from_sim no)
 		(at 140.97 73.66 0)

Commit message: ready for last scrut
Parts:
- removed C8: 47p 50V C0G, 0_capacitor_smd:C_0402_1005Metric, symbol Device:C
Changed lines of the file:
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@@
-	)
-	(junction
-		(at 154.94 53.34)
-		(diameter 0)
-		(color 0 0 0 0)
 	)
 	(junction
@@
 	(junction
 		(at 77.47 53.34)
-		(diameter 0)
-		(color 0 0 0 0)
-	)
-	(junction
-		(at 154.94 69.85)
 		(diameter 0)
 		(color 0 0 0 0)
@@
 	(wire
 		(pts
-			(xy 125.73 69.85) (xy 154.94 69.85)
-		)
-		(stroke
-			(width 0)
-			(type default)
-		)
-	)
-	(wire
-		(pts
 			(xy 125.73 73.66) (xy 133.35 73.66)
 		)
@@
 	(wire
 		(pts
-			(xy 154.94 69.85) (xy 170.18 69.85)
+			(xy 125.73 69.85) (xy 170.18 69.85)
 		)
 		(stroke
@@
 	(wire
 		(pts
-			(xy 154.94 63.5) (xy 154.94 69.85)
-		)
-		(stroke
-			(width 0)
-			(type default)
-		)
-	)
-	(wire
-		(pts
 			(xy 170.18 85.09) (xy 170.18 95.25)
 		)
@@
 	(wire
 		(pts
-			(xy 152.4 53.34) (xy 154.94 53.34)
+			(xy 152.4 53.34) (xy 170.18 53.34)
 		)
 		(stroke
@@
 	(wire
 		(pts
-			(xy 154.94 53.34) (xy 170.18 53.34)
-		)
-		(stroke
-			(width 0)
-			(type default)
-		)
-	)
-	(wire
-		(pts
 			(xy 125.73 53.34) (xy 137.16 53.34)
 		)
@@
 		(pts
 			(xy 224.79 53.34) (xy 236.22 53.34)
-		)
-		(stroke
-			(width 0)
-			(type default)
-		)
-	)
-	(wire
-		(pts
-			(xy 154.94 53.34) (xy 154.94 55.88)
 		)
 		(stroke
@@
 		)
 	)
-	(symbol
-		(lib_id "Device:C")
-		(at 154.94 59.69 0)
-		(unit 1)
-		(exclude_from_sim no)
-		(in_bom yes)
-		(on_board yes)
-		(dnp no)
-		(fields_autoplaced yes)
-		(property "Reference" "C8"
-			(at 158.75 59.0549 0)
-			(effects
-				(font
-					(size 1.27 1.27)
-				)
-				(justify left)
-			)
-		)
-		(property "Value" "47p 50V C0G"
-			(at 158.75 60.96 0)
-			(effects
-				(font
-					(size 0.762 0.762)
-				)
-				(justify left)
-			)
-		)
-		(property "Footprint" "0_capacitor_smd:C_0402_1005Metric"
-			(at 155.9052 63.5 0)
-			(effects
-				(font
-					(size 1.27 1.27)
-				)
-				(hide yes)
-			)
-		)
-		(property "Datasheet" "~"
-			(at 154.94 59.69 0)
-			(effects
-				(font
-					(size 1.27 1.27)
-				)
-				(hide yes)
-			)
-		)
-		(property "Description" "Unpolarized capacitor"
-			(at 154.94 59.69 0)
-			(effects
-				(font
-					(size 1.27 1.27)
-				)
-				(hide yes)
-			)
-		)
-		(property "LCSC" "C1567"
-			(at 154.94 59.69 0)
-			(effects
-				(font
-					(size 1.27 1.27)
-				)
-				(hide yes)
-			)
-		)
-		(property "Name" ""
-			(at 154.94 59.69 0)
-			(effects
-				(font
-					(size 1.27 1.27)
-				)
-				(hide yes)
-			)
-		)
-		(pin "2"
-		)
-		(pin "1"
-		)
-		(instances
-			(project "fdcanhat"
-				(path "/4375c315-c696-43df-ab5b-868bd3f1287b/62df980a-c264-4c67-968f-e32163c54c0c"
-					(reference "C8")
-					(unit 1)
-				)
-			)
-		)
-	)
