File: fdcanhat/voltage_measurement.kicad_sch (KiCad schematic)
At the start: 6 parts, among them U9 ADS1115IDGSR

Commit message: board layout done, ready for routing
Parts:
- C41: value 1u 50V X7R -> 1u 50V X5R; footprint 0_capacitor_smd:C_0402_1005Metric -> 0_capacitor_smd:C_0603_1608Metric; LCSC C307331 -> C15849
- renumbered C40 to C42, R16 to R19, R14 to R20, R15 to R21, U9 to U10
Connections:
- net SCL renamed MON_SCL
- net SDA renamed MON_SDA
Changed lines of the file:
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@@
 		)
 	)
-	(hierarchical_label "SCL"
+	(hierarchical_label "MON_SCL"
 		(shape input)
 		(at 66.04 86.36 180)
@@
 		)
 	)
-	(hierarchical_label "SDA"
+	(hierarchical_label "MON_SDA"
 		(shape bidirectional)
 		(at 66.04 83.82 180)
@@
 		(on_board yes)
 		(dnp no)
-		(property "Reference" "C40"
+		(property "Reference" "C42"
 			(at 110.49 58.42 0)
 			(effects
@@
 			(project "fdcanhat"
 				(path "/4375c315-c696-43df-ab5b-868bd3f1287b/fa34ba4e-0a0d-40f6-bbb7-8a98a9ddd90d"
-					(reference "C40")
+					(reference "C42")
 					(unit 1)
 				)
@@
 		(dnp no)
 		(fields_autoplaced yes)
-		(property "Reference" "#PWR059"
+		(property "Reference" "#PWR079"
 			(at 121.92 58.42 0)
 			(effects
@@
 			(project "fdcanhat"
 				(path "/4375c315-c696-43df-ab5b-868bd3f1287b/fa34ba4e-0a0d-40f6-bbb7-8a98a9ddd90d"
-					(reference "#PWR059")
+					(reference "#PWR079")
 					(unit 1)
 				)
@@
 			)
 		)
-		(property "Value" "1u 50V X7R"
+		(property "Value" "1u 50V X5R"
 			(at 97.79 63.5 0)
 			(effects
@@
 			)
 		)
-		(property "Footprint" "0_capacitor_smd:C_0402_1005Metric"
+		(property "Footprint" "0_capacitor_smd:C_0603_1608Metric"
 			(at 98.7552 64.77 0)
 			(effects
@@
 			)
 		)
-		(property "LCSC" "C307331"
+		(property "LCSC" "C15849"
 			(at 97.79 60.96 0)
 			(effects
@@
 		(dnp no)
 		(fields_autoplaced yes)
-		(property "Reference" "#PWR058"
+		(property "Reference" "#PWR082"
 			(at 142.24 104.14 0)
 			(effects
@@
 			(project "fdcanhat"
 				(path "/4375c315-c696-43df-ab5b-868bd3f1287b/fa34ba4e-0a0d-40f6-bbb7-8a98a9ddd90d"
-					(reference "#PWR058")
+					(reference "#PWR082")
 					(unit 1)
 				)
@@
 		(dnp no)
 		(fields_autoplaced yes)
-		(property "Reference" "#PWR060"
+		(property "Reference" "#PWR081"
 			(at 110.49 74.93 0)
 			(effects
@@
 			(project "fdcanhat"
 				(path "/4375c315-c696-43df-ab5b-868bd3f1287b/fa34ba4e-0a0d-40f6-bbb7-8a98a9ddd90d"
-					(reference "#PWR060")
+					(reference "#PWR081")
 					(unit 1)
 				)
@@
 		(dnp no)
 		(fields_autoplaced yes)
-		(property "Reference" "R15"
+		(property "Reference" "R21"
 			(at 88.9 74.2949 0)
 			(effects
@@
 			(project "fdcanhat"
 				(path "/4375c315-c696-43df-ab5b-868bd3f1287b/fa34ba4e-0a0d-40f6-bbb7-8a98a9ddd90d"
-					(reference "R15")
+					(reference "R21")
 					(unit 1)
 				)
@@
 		(dnp no)
 		(fields_autoplaced yes)
-		(property "Reference" "R14"
+		(property "Reference" "R20"
 			(at 78.74 74.2949 0)
 			(effects
@@
 			(project "fdcanhat"
 				(path "/4375c315-c696-43df-ab5b-868bd3f1287b/fa34ba4e-0a0d-40f6-bbb7-8a98a9ddd90d"
-					(reference "R14")
+					(reference "R20")
 					(unit 1)
 				)
@@
 		(dnp no)
 		(fields_autoplaced yes)
-		(property "Reference" "U9"
+		(property "Reference" "U10"
 			(at 142.24 63.5 0)
 			(effects
@@
 			(project ""
 				(path "/4375c315-c696-43df-ab5b-868bd3f1287b/fa34ba4e-0a0d-40f6-bbb7-8a98a9ddd90d"
-					(reference "U9")
+					(reference "U10")
 					(unit 1)
 				)
@@
 		(dnp no)
 		(fields_autoplaced yes)
-		(property "Reference" "#PWR061"
+		(property "Reference" "#PWR080"
 			(at 97.79 74.93 0)
 			(effects
@@
 			(project "fdcanhat"
 				(path "/4375c315-c696-43df-ab5b-868bd3f1287b/fa34ba4e-0a0d-40f6-bbb7-8a98a9ddd90d"
-					(reference "#PWR061")
+					(reference "#PWR080")
 					(unit 1)
 				)
@@
 		(dnp no)
 		(fields_autoplaced yes)
-		(property "Reference" "R16"
+		(property "Reference" "R19"
 			(at 119.38 71.7549 0)
 			(effects
@@
 			(project "fdcanhat"
 				(path "/4375c315-c696-43df-ab5b-868bd3f1287b/fa34ba4e-0a0d-40f6-bbb7-8a98a9ddd90d"
-					(reference "R16")
-					(unit 1)
-				)
+					(reference "R19")
+					(unit 1)
+				)

Commit message: almost done
Parts:
- renumbered C41 to C35, C42 to C36, R19 to R15, R20 to R16, R21 to R17, U10 to U9
Connections:
- net +5V_VMON: now also U9.6 (AIN2); no longer U9.4 (AIN0)
- net +BAT_IMON: now also U9.4 (AIN0); no longer U9.6 (AIN2)
Changed lines of the file:
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@@
+		)
+	)
+	(hierarchical_label "+BAT_IMON"
+		(shape input)
+		(at 177.8 71.12 0)
+		(effects
+			(font
+				(size 1.27 1.27)
+			)
+			(justify left)
 		)
 	)
@@
 		)
 	)
-	(hierarchical_label "+5V_VMON"
-		(shape input)
-		(at 177.8 71.12 0)
-		(effects
-			(font
-				(size 1.27 1.27)
-			)
-			(justify left)
-		)
-	)
-	(hierarchical_label "+BAT_IMON"
-		(shape input)
-		(at 177.8 81.28 0)
-		(effects
-			(font
-				(size 1.27 1.27)
-			)
-			(justify left)
-		)
-	)
 	(hierarchical_label "+BAT_PROT_VMON"
 		(shape input)
@@
 		)
 	)
+	(hierarchical_label "+5V_VMON"
+		(shape input)
+		(at 177.8 81.28 0)
+		(effects
+			(font
+				(size 1.27 1.27)
+			)
+			(justify left)
+		)
+	)
 	(symbol
 		(lib_id "Device:C")
@@
 		(on_board yes)
 		(dnp no)
-		(property "Reference" "C42"
+		(property "Reference" "C36"
 			(at 110.49 58.42 0)
 			(effects
@@
 			)
 		)
+		(property "Name" ""
+			(at 110.49 60.96 0)
+			(effects
+				(font
+					(size 1.27 1.27)
+				)
+				(hide yes)
+			)
+		)
 		(pin "2"
 		)
@@
 			(project "fdcanhat"
 				(path "/4375c315-c696-43df-ab5b-868bd3f1287b/fa34ba4e-0a0d-40f6-bbb7-8a98a9ddd90d"
-					(reference "C42")
+					(reference "C36")
 					(unit 1)
 				)
@@
 		(dnp no)
 		(fields_autoplaced yes)
-		(property "Reference" "#PWR079"
+		(property "Reference" "#PWR080"
 			(at 121.92 58.42 0)
 			(effects
@@
 			(project "fdcanhat"
 				(path "/4375c315-c696-43df-ab5b-868bd3f1287b/fa34ba4e-0a0d-40f6-bbb7-8a98a9ddd90d"
-					(reference "#PWR079")
+					(reference "#PWR080")
 					(unit 1)
 				)
@@
 		(on_board yes)
 		(dnp no)
-		(property "Reference" "C41"
+		(property "Reference" "C35"
 			(at 97.79 58.42 0)
 			(effects
@@
 			)
 		)
+		(property "Name" ""
+			(at 97.79 60.96 0)
+			(effects
+				(font
+					(size 1.27 1.27)
+				)
+				(hide yes)
+			)
+		)
 		(pin "2"
 		)
@@
 			(project "fdcanhat"
 				(path "/4375c315-c696-43df-ab5b-868bd3f1287b/fa34ba4e-0a0d-40f6-bbb7-8a98a9ddd90d"
-					(reference "C41")
+					(reference "C35")
 					(unit 1)
 				)
@@
 		(dnp no)
 		(fields_autoplaced yes)
-		(property "Reference" "#PWR082"
+		(property "Reference" "#PWR083"
 			(at 142.24 104.14 0)
 			(effects
@@
 			(project "fdcanhat"
 				(path "/4375c315-c696-43df-ab5b-868bd3f1287b/fa34ba4e-0a0d-40f6-bbb7-8a98a9ddd90d"
-					(reference "#PWR082")
+					(reference "#PWR083")
 					(unit 1)
 				)
@@
 		(dnp no)
 		(fields_autoplaced yes)
-		(property "Reference" "#PWR081"
+		(property "Reference" "#PWR082"
 			(at 110.49 74.93 0)
 			(effects
@@
 			(project "fdcanhat"
 				(path "/4375c315-c696-43df-ab5b-868bd3f1287b/fa34ba4e-0a0d-40f6-bbb7-8a98a9ddd90d"
-					(reference "#PWR081")
+					(reference "#PWR082")
 					(unit 1)
 				)
@@
 		(dnp no)
 		(fields_autoplaced yes)
-		(property "Reference" "R21"
+		(property "Reference" "R17"
 			(at 88.9 74.2949 0)
 			(effects
@@
 			)
 		)
+		(property "Name" ""
+			(at 86.36 74.93 0)
+			(effects
+				(font
+					(size 1.27 1.27)
+				)
+				(hide yes)
+			)
+		)
 		(pin "1"
 		)
@@
 			(project "fdcanhat"
 				(path "/4375c315-c696-43df-ab5b-868bd3f1287b/fa34ba4e-0a0d-40f6-bbb7-8a98a9ddd90d"
-					(reference "R21")
+					(reference "R17")
 					(unit 1)
 				)
@@
 		(dnp no)
 		(fields_autoplaced yes)
-		(property "Reference" "R20"
+		(property "Reference" "R16"
 			(at 78.74 74.2949 0)
 			(effects
@@
 			)
 		)
+		(property "Name" ""
+			(at 76.2 74.93 0)
+			(effects
+				(font
+					(size 1.27 1.27)
+				)
+				(hide yes)
+			)
+		)
 		(pin "1"
 		)
@@
 			(project "fdcanhat"
 				(path "/4375c315-c696-43df-ab5b-868bd3f1287b/fa34ba4e-0a0d-40f6-bbb7-8a98a9ddd90d"
-					(reference "R20")
+					(reference "R16")
 					(unit 1)
 				)
@@
 		(dnp no)
 		(fields_autoplaced yes)
-		(property "Reference" "U10"
+		(property "Reference" "U9"
 			(at 142.24 63.5 0)
 			(effects
@@
 			)
 		)
+		(property "Name" ""
+			(at 142.24 68.58 0)
+			(effects
+				(font
+					(size 1.27 1.27)
+				)
+				(hide yes)
+			)
+		)
 		(pin "7"
 		)
@@
 			(project ""
 				(path "/4375c315-c696-43df-ab5b-868bd3f1287b/fa34ba4e-0a0d-40f6-bbb7-8a98a9ddd90d"
-					(reference "U10")
+					(reference "U9")
 					(unit 1)
 				)
@@
 		(dnp no)
 		(fields_autoplaced yes)
-		(property "Reference" "#PWR080"
+		(property "Reference" "#PWR081"
 			(at 97.79 74.93 0)
 			(effects
@@
 			(project "fdcanhat"
 				(path "/4375c315-c696-43df-ab5b-868bd3f1287b/fa34ba4e-0a0d-40f6-bbb7-8a98a9ddd90d"
-					(reference "#PWR080")
+					(reference "#PWR081")
 					(unit 1)
 				)
@@
 		(dnp no)
 		(fields_autoplaced yes)
-		(property "Reference" "R19"
+		(property "Reference" "R15"
 			(at 119.38 71.7549 0)
 			(effects
@@
 			)
 		)
+		(property "Name" ""
+			(at 116.84 72.39 0)
+			(effects
+				(font
+					(size 1.27 1.27)
+				)
+				(hide yes)
+			)
+		)
 		(pin "1"
 		)
@@
 			(project "fdcanhat"
 				(path "/4375c315-c696-43df-ab5b-868bd3f1287b/fa34ba4e-0a0d-40f6-bbb7-8a98a9ddd90d"
-					(reference "R19")
-					(unit 1)
-				)
+					(reference "R15")
+					(unit 1)
+				)

Commit message: ready for last scrut
Parts:
- C35: value 1u 50V X5R -> 1u 25V X7R; footprint 0_capacitor_smd:C_0603_1608Metric -> 0_capacitor_smd:C_0402_1005Metric; LCSC C15849 -> C52923
Changed lines of the file:
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@@
 			)
 		)
-		(property "Value" "1u 50V X5R"
+		(property "Value" "1u 25V X7R"
 			(at 97.79 63.5 0)
 			(effects
@@
 			)
 		)
-		(property "Footprint" "0_capacitor_smd:C_0603_1608Metric"
+		(property "Footprint" "0_capacitor_smd:C_0402_1005Metric"
 			(at 98.7552 64.77 0)
 			(effects
@@
 			)
 		)
-		(property "LCSC" "C15849"
+		(property "LCSC" "C52923"
 			(at 97.79 60.96 0)
 			(effects

Commit message: sent to production
Connections:
- net +3V3: now also U9.7 (AIN3)
- no-connect marks 1 -> 0
Changed lines of the file:
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@@
 		(color 0 0 0 0)
 	)
-	(no_connect
-		(at 154.94 86.36)
-	)
 	(wire
 		(pts
@@
 	(wire
 		(pts
+			(xy 154.94 86.36) (xy 201.93 86.36)
+		)
+		(stroke
+			(width 0)
+			(type default)
+		)
+	)
+	(wire
+		(pts
 			(xy 66.04 83.82) (xy 76.2 83.82)
 		)
@@
 		(pts
 			(xy 97.79 64.77) (xy 97.79 68.58)
+		)
+		(stroke
+			(width 0)
+			(type default)
+		)
+	)
+	(wire
+		(pts
+			(xy 201.93 86.36) (xy 201.93 85.09)
 		)
 		(stroke
@@
 					(unit 1)
 				)
+			)
+		)
+	)
+	(symbol
+		(lib_id "power:+3.3V")
+		(at 201.93 85.09 0)
+		(unit 1)
+		(exclude_from_sim no)
+		(in_bom yes)
+		(on_board yes)
+		(dnp no)
+		(fields_autoplaced yes)
+		(property "Reference" "#PWR019"
+			(at 201.93 88.9 0)
+			(effects
+				(font
+					(size 1.27 1.27)
+				)
+				(hide yes)
+			)
+		)
+		(property "Value" "+3V3"
+			(at 201.93 80.01 0)
+			(effects
+				(font
+					(size 1.27 1.27)
+				)
+			)
+		)
+		(property "Footprint" ""
+			(at 201.93 85.09 0)
+			(effects
+				(font
+					(size 1.27 1.27)
+				)
+				(hide yes)
+			)
+		)
+		(property "Datasheet" ""
+			(at 201.93 85.09 0)
+			(effects
+				(font
+					(size 1.27 1.27)
+				)
+				(hide yes)
+			)
+		)
+		(property "Description" "Power symbol creates a global label with name \"+3.3V\""
+			(at 201.93 85.09 0)
+			(effects
+				(font
+					(size 1.27 1.27)
+				)
+				(hide yes)
+			)
+		)
+		(pin "1"
+		)
+		(instances
+			(project "fdcanhat"
+				(path "/4375c315-c696-43df-ab5b-868bd3f1287b/fa34ba4e-0a0d-40f6-bbb7-8a98a9ddd90d"
+					(reference "#PWR019")
+					(unit 1)
+				)
